File: pcb/pcb.kicad_sch (KiCad schematic)
At the start: 5 parts, among them U1 xiao-ble

Commit message: v2
Parts:
- added J2: Conn_01x04_Socket, lego:voltage-converter, symbol Connector:Conn_01x04_Socket
- added Motor3, Motor4: Conn_01x04_Female, Connector_JST:JST_XH_S4B-XH-A_1x04_P2.50mm_Horizontal, symbol Connector:Conn_01x04_Female
- added SW1: SW_SPDT, Connector_PinHeader_2.54mm:PinHeader_1x03_P2.54mm_Vertical, symbol Switch:SW_SPDT
- added TB2: TB6612_Breakout, lego:TB6612-breakout, symbol lego:TB6612_Breakout
- J1: renamed from Batt1; value Conn_01x04_Female -> Conn_01x02_Socket; footprint Connector_JST:JST_XH_S4B-XH-A_1x04_P2.50mm_Horizontal -> Connector_PinHeader_2.54mm:PinHeader_1x02_P2.54mm_Vertical; symbol Connector:Conn_01x04_Female -> Connector:Conn_01x02_Socket
- TB1: footprint lego:Breakout-16_17.8x20.3mm -> lego:TB6612-breakout
- U1: value xiao-ble -> MCU_xiao-ble; footprint lego:xiao-ble-tht -> zzkeeb:MCU_xiao-ble-smd; symbol kleeb-mcu:xiao-ble -> zzkeeb:MCU_xiao-ble
Connections:
- net +3.3V: now also J2.3 (Pin_3), TB2.15 (VCC); no longer U1.19 (BAT)
- net +9V: now also J2.1 (Pin_1), Motor3.1 (Pin_1), Motor4.1 (Pin_1), SW1.1 (A), TB2.16 (VM); no longer J1.1 (Pin_1)
- net GND: now also J1.2 (Pin_2), J2.2 (Pin_2), J2.4 (Pin_4), Motor3.4 (Pin_4), Motor4.4 (Pin_4), TB2.14 (GND), TB2.8 (GND), TB2.9 (GND); no longer J1.4 (Pin_4)
- net STBY: now also U1.1 (A2/0.02_H), TB2.4 (STBY); no longer U1.4 (A11/0.29)
- net AIN1_2: now reaches U1.10 (A5_MISO/1.14)
- net AIN1_2: now also TB2.3 (AIN1)
- net AIN2_2: now reaches U1.11 (A6_MOSI/1.15)
- net AIN2_2: now also TB2.2 (AIN2)
- net BIN1_2: now reaches U1.21 (NFC1/0.09_H)
- net BIN1_2: now also TB2.5 (BIN1)
- net BIN2_2: now reaches U1.22 (NFC2/0.10_H)
- net BIN2_2: now also TB2.6 (BIN2)
- net BIN1_1: now reaches U1.8 (B9_RX/1.12)
- net BIN1_1: now also TB1.5 (BIN1)
- net BIN2_1: now reaches U1.9 (A7_SCK/1.13)
- net BIN2_1: now also TB1.6 (BIN2)
- net A01 renamed A01_1
- net A01_1: now also Motor1.2 (Pin_2); no longer Motor2.3 (Pin_3)
- net A02 renamed A02_1
- net A02_1: now also Motor1.3 (Pin_3); no longer Motor2.2 (Pin_2)
- net AIN1 renamed AIN1_1
- net AIN1_1: now also U1.6 (A9_SCL/0.05_H); no longer U1.5 (A8_SDA/0.04_H)
- net AIN2 renamed AIN2_1
- net AIN2_1: now also U1.7 (B8_TX/1.11); no longer U1.6 (A9_SCL/0.05_H)
- net B01 renamed B01_1
- net B01_1: now also Motor2.2 (Pin_2); no longer Motor1.2 (Pin_2)
- net B02 renamed B02_1
- net B02_1: now also Motor2.3 (Pin_3); no longer Motor1.3 (Pin_3)
- net BIN1 renamed PWMB_1
- net PWMB_1: now also TB1.7 (PWMB); no longer TB1.5 (BIN1)
- net BIN2 renamed PWMA_1
- net PWMA_1: now also TB1.1 (PWMA); no longer TB1.6 (BIN2)
- removed net PWMA: TB1.1 (PWMA), U1.7 (B8_TX/1.11)
- removed net PWMB: TB1.7 (PWMB), U1.1 (A2/0.02_H)
- new net A01_2: Motor3.2 (Pin_2), TB2.13 (A01)
- new net A02_2: Motor3.3 (Pin_3), TB2.12 (A02)
- new net B01_2: Motor4.2 (Pin_2), TB2.10 (B01)
- new net B02_2: Motor4.3 (Pin_3), TB2.11 (B02)
- new net BAT: J1.1 (Pin_1), SW1.2 (B)
- new net PWMA_2: TB2.1 (PWMA), U1.4 (A11/0.29)
- new net PWMB_2: TB2.7 (PWMB), U1.5 (A8_SDA/0.04_H)
- no-connect marks 12 -> 6
Other:
- moved on the sheet: Motor1, Motor2
